File: KiCAD/BMT BionX_Minimum_Translator.sch (KiCad schematic (older format))
At the start: 34 parts

Commit message: Add files via upload
Parts:
- removed C? (x2): 10µ, symbol Device:CP
- removed C?: 47µ, symbol Device:CP
- removed D?: D_Zener 4.7V, symbol Device:D_Zener
- removed J?: External BB Torquesensor, symbol Connector:Conn_01x04_Male
- removed J?: Light output, symbol Connector:Conn_01x02_Female
- removed Q?: IRF6644, Package_DirectFET:DirectFET_MN, symbol Transistor_FET:IRF6644
- removed R? (x2): 56k, symbol Device:R
- removed R?: 4,7k, symbol Device:R
- removed R?: 2.2k, symbol Device:R
- removed R?: 1k, symbol Device:R
- removed R?: 22k, symbol Device:R
- removed SW?: SW_DPST_x2, symbol Switch:SW_DPST_x2
- removed U?: StepDown 5V, Package_TO_SOT_THT:TO-220-5_P3.4x3.7mm_StaggerOdd_Lead3.8mm_Vertical, symbol Regulator_Switching:LM2595T-5
- removed U?: StepDown 6V, Package_TO_SOT_THT:TO-220-5_P3.4x3.7mm_StaggerOdd_Lead3.8mm_Vertical, symbol Regulator_Switching:LM2595T-12
- removed U?: ACS712xLCTR-05B, Package_SO:SOIC-8_3.9x4.9mm_P1.27mm, symbol Sensor_Current:ACS712xLCTR-05B
- removed U?: BTS432, Package_TO_SOT_SMD:TO-263-7_TabPin4, symbol Power_Management:BTS432
- added C?: 100 nF, symbol Device:C
- added C?: 10 uF, symbol Device:CP
- added Q?: BD139, Package_TO_SOT_THT:TO-126-3_Vertical, symbol Transistor_BJT:BD139
- added R?: 30, symbol Device:R
- added U?: LM7805_TO220, Package_TO_SOT_THT:TO-220-3_Vertical, symbol Regulator_Linear:LM7805_TO220
- R?: value 56k -> 1k
- R?: value 2.2k -> 2k2
Connections:
- net labels removed: -BATT
- wire segments 209 -> 121
Other:
- note removed: "Antiblitzschaltung optional für Akkus ohne Schalter am BMS"
- moved on the sheet: C?, J?, R?
